Commit message: Update differential_drive_bot.urdf
Updated the urdf so that it can move in willow garage world in gazebo

File: urdf/differential_drive_bot.urdf (robot description, URDF)
Before this commit: robot test_robot, 6 links, 5 joints
Links:
- link scanner: mass 0.03 -> 0.000001; geometry collision box size=0.015 0.045 0.015; visual box size=0.05 0.05 0.05
